File: xdevrf03/xdevrf03.kicad_pcb (KiCad board)
At the start: 4 copper layers, 50.8 x 22.9 mm, 20 parts, among them P1 USB_C_Plug_USB2.0, SW1 RST, SW2 BOOT, U1 AP2112K-3.3, U2 Feather, U3 ESP32-C3-MINI-1

Commit message: Schematic updates and pcb silkscreen
Parts:
- added G***: LOGO, symbols:logo-bsilk, F.Cu at (132.7, 94.9)
Other:
- board text added: "esp32-c3-mini-1"
- board text added: "xdevrf03 :: Rev A nnarain"
