File: xdevrf03/xdevrf03.kicad_sch (KiCad schematic)
At the start: 19 parts, among them P1 USB_C_Plug_USB2.0, SW1 RST, SW2 BOOT, U1 AP2112K-3.3, U2 Feather, U3 ESP32-C3-MINI-1

Commit message: Schematic updates and pcb silkscreen
Parts:
- SW1, SW2: LCSC (none) -> C720477
- U1: LCSC (none) -> C51118
Changed lines of the file:
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@@
+      (effects (font (size 1.27 1.27)) hide)
+    )
+    (property "LCSC" "C720477" (id 4) (at 36.83 91.44 90)
       (effects (font (size 1.27 1.27)) hide)
     )
@@
       (effects (font (size 1.27 1.27)) hide)
     )
+    (property "LCSC" "C51118" (id 4) (at 68.58 25.4 0)
+      (effects (font (size 1.27 1.27)) hide)
+    )
     (pin "1")
     (pin "2")
@@
       (effects (font (size 1.27 1.27)) hide)
     )
+    (property "LCSC" "C720477" (id 4) (at 59.69 91.44 90)
+      (effects (font (size 1.27 1.27)) hide)
+    )
